File: Programmer.sch (KiCad schematic (older format))
At the start: 38 parts, among them J1 USB_C_Receptacle_USB2.0, J2 Conn_02x08_Top_Bottom, J3 Conn_02x08_Top_Bottom, U2 93LCxxC, U3 NCP1117-3.3, U4 FT2232H, Y1 12MHz

Commit message: Revision B
Parts:
- removed J2, J3: Conn_02x08_Top_Bottom, Connector_PinHeader_2.54mm:PinHeader_2x08_P2.54mm_Vertical, symbol Connector_Generic:Conn_02x08_Top_Bottom
- added J2: Conn_01x04, Connector_PinHeader_2.54mm:PinHeader_1x04_P2.54mm_Vertical, symbol Connector_Generic:Conn_01x04
- added J3: Conn_01x02, Connector_PinHeader_2.54mm:PinHeader_1x02_P2.54mm_Vertical, symbol Connector_Generic:Conn_01x02
Connections:
- net +5V: now reaches J1.A4 (VBUS), J1.A9 (VBUS), J1.B4 (VBUS), J1.B9 (VBUS), U3.3 (VI)
- net at U4.16 (ADBUS0): now also J2.1 (Pin_1)
- net at U4.17 (ADBUS1): now also J2.2 (Pin_2)
- net at U4.18 (ADBUS2): now also J2.3 (Pin_3)
- net at U4.19 (ADBUS3): now also J2.4 (Pin_4)
- net at U4.38 (BDBUS0): now also J3.1 (Pin_1)
- net at U4.39 (BDBUS1): now also J3.2 (Pin_2)
- no-connect marks 3 -> 26
Other:
- moved on the sheet: D2, D3, J1, R11, R3, R4, U3
